File: lets_split/lets_split.sch (KiCad schematic (older format))
At the start: 60 parts, among them J1 3PIN, J2 6PIN, J3 3PIN, SW1 SW_PUSH, SW10 SW_PUSH, SW11 SW_PUSH, SW12 SW_PUSH, SW13 SW_PUSH, SW14 SW_PUSH, SW15 SW_PUSH, SW16 SW_PUSH, SW17 SW_PUSH, SW18 SW_PUSH, SW19 SW_PUSH, SW2 SW_PUSH, SW20 SW_PUSH, SW21 SW_PUSH, SW22 SW_PUSH, SW23 SW_PUSH, SW24 SW_PUSH, SW3 SW_PUSH, SW4 SW_PUSH, SW5 SW_PUSH, SW6 SW_PUSH, SW7 SW_PUSH, SW8 SW_PUSH, SW9 SW_PUSH, U1 TEENSY2.0, U2 HOLE, U3 HOLE, U4 HOLE, U5 HOLE

Commit message: Rev 1 complete
Parts:
- removed D10, D11, D12, D13, D14, D15, D16, D17, D18, D19, D2, D20, D21, D22, D23, D24, D3, D4, D5, D6, D7, D8, D9: D, Diodes_ThroughHole:Diode_DO-41_SOD81_Horizontal_RM10, symbol D
- removed R1, R2: R, footprint:RESISTOR, symbol R
- removed U1: TEENSY2.0, footprint:TEENSY_2.0, symbol TEENSY2.0
- removed W1: TEST, prettylib:JUMPER_SMD_2DUB, symbol TEST
- added D1, D2: Inolux_IN-PI554FCH, LED_SMD:LED_Inolux_IN-PI554FCH_PLCC4_5.0x5.0mm_P3.2mm, symbol LED:Inolux_IN-PI554FCH
- added D10, D11, D12, D13, D14, D15, D16, D17, D18, D19, D20, D21, D22, D23, D24, D25, D26, D4, D5, D6, D7, D8, D9: D, LetsSplitSingle:D_DO-41_SOD81_P10.16mm_Horizontal, symbol lets_split-rescue:D-lets_split-rescue
- added J1: Pro Micro 5V, LetsSplitSingle:Pro_Micro, symbol Connector_Generic:Conn_02x12_Counter_Clockwise
- added JP1: Jumper, Jumper:SolderJumper-2_P1.3mm_Open_TrianglePad1.0x1.5mm, symbol Device:Jumper
- added SW1, SW22: Rotary_Encoder_Switch, Rotary_Encoder:RotaryEncoder_Alps_EC12E-Switch_Vertical_H20mm, symbol Device:Rotary_Encoder_Switch
- D3: renamed from D1; footprint Diodes_ThroughHole:Diode_DO-41_SOD81_Horizontal_RM10 -> LetsSplitSingle:D_DO-41_SOD81_P10.16mm_Horizontal; symbol D -> lets_split-rescue:D-lets_split-rescue
- J2: renamed from J1; footprint prettylib:jumper -> LetsSplitSingle:3_pin_TP; symbol 3PIN -> lets_split-rescue:3PIN-lets_split-rescue
- J3: renamed from J2; footprint footprint:4pin35mmAudio -> LetsSplitSingle:4pin35mmAudio; symbol 6PIN -> lets_split-rescue:6PIN-lets_split-rescue
- J4: renamed from J3; footprint prettylib:jumper -> LetsSplitSingle:3_pin_TP; symbol 3PIN -> lets_split-rescue:3PIN-lets_split-rescue
- SW10: renamed from SW9; symbol SW_PUSH -> lets_split-rescue:SW_PUSH-lets_split-rescue
- SW11: renamed from SW10; symbol SW_PUSH -> lets_split-rescue:SW_PUSH-lets_split-rescue
- SW12: renamed from SW11; symbol SW_PUSH -> lets_split-rescue:SW_PUSH-lets_split-rescue
- SW13: renamed from SW12; symbol SW_PUSH -> lets_split-rescue:SW_PUSH-lets_split-rescue
- SW14: renamed from SW13; symbol SW_PUSH -> lets_split-rescue:SW_PUSH-lets_split-rescue
- SW15: renamed from SW14; symbol SW_PUSH -> lets_split-rescue:SW_PUSH-lets_split-rescue
- SW16: renamed from SW15; symbol SW_PUSH -> lets_split-rescue:SW_PUSH-lets_split-rescue
- SW17: renamed from SW16; symbol SW_PUSH -> lets_split-rescue:SW_PUSH-lets_split-rescue
- SW18: renamed from SW17; symbol SW_PUSH -> lets_split-rescue:SW_PUSH-lets_split-rescue
- SW19: renamed from SW18; symbol SW_PUSH -> lets_split-rescue:SW_PUSH-lets_split-rescue
- SW2: renamed from SW1; symbol SW_PUSH -> lets_split-rescue:SW_PUSH-lets_split-rescue
- SW20: renamed from SW19; symbol SW_PUSH -> lets_split-rescue:SW_PUSH-lets_split-rescue
- SW21: renamed from SW20; symbol SW_PUSH -> lets_split-rescue:SW_PUSH-lets_split-rescue
- SW23: renamed from SW21; symbol SW_PUSH -> lets_split-rescue:SW_PUSH-lets_split-rescue
- SW24: renamed from SW22; symbol SW_PUSH -> lets_split-rescue:SW_PUSH-lets_split-rescue
- SW25: renamed from SW23; symbol SW_PUSH -> lets_split-rescue:SW_PUSH-lets_split-rescue
- SW26: renamed from SW24; symbol SW_PUSH -> lets_split-rescue:SW_PUSH-lets_split-rescue
- SW3: renamed from SW2; symbol SW_PUSH -> lets_split-rescue:SW_PUSH-lets_split-rescue
- SW4: renamed from SW3; symbol SW_PUSH -> lets_split-rescue:SW_PUSH-lets_split-rescue
- SW5: renamed from SW4; symbol SW_PUSH -> lets_split-rescue:SW_PUSH-lets_split-rescue
- SW6: renamed from SW5; symbol SW_PUSH -> lets_split-rescue:SW_PUSH-lets_split-rescue
- SW7: renamed from SW6; symbol SW_PUSH -> lets_split-rescue:SW_PUSH-lets_split-rescue
- SW8: renamed from SW7; symbol SW_PUSH -> lets_split-rescue:SW_PUSH-lets_split-rescue
- SW9: renamed from SW8; symbol SW_PUSH -> lets_split-rescue:SW_PUSH-lets_split-rescue
- U1: renamed from U3; footprint prettylib:HOLE -> LetsSplitSingle:LS_HOLE; symbol HOLE -> lets_split-rescue:HOLE-lets_split-rescue
- U2, U4: footprint prettylib:HOLE -> LetsSplitSingle:LS_HOLE; symbol HOLE -> lets_split-rescue:HOLE-lets_split-rescue
- U3: renamed from U5; footprint prettylib:HOLE -> LetsSplitSingle:LS_HOLE; symbol HOLE -> lets_split-rescue:HOLE-lets_split-rescue
- W1: renamed from W2; footprint Wire_Pads:SolderWirePad_single_2mmDrill -> TestPoint:TestPoint_Plated_Hole_D2.0mm; symbol TEST_1P -> lets_split-rescue:TEST_1P-lets_split-rescue
Connections:
- net labels added: EncA, EncB
- wire segments 24 -> 68
- no-connect marks 0 -> 7
